File: Debug_subsystem.sch (KiCad schematic (older format))
At the start: 2 parts

Commit message: This is a new commit.
Parts:
- gave numbers to parts that had none: 2
Changed lines of the file:
@@
 $EndDescr
 $Comp
-L Connector:Conn_ARM_JTAG_SWD_10 J?
+L Connector:Conn_ARM_JTAG_SWD_10 J1
 U 1 1 614AA0C1
 P 5150 3550
-F 0 "J?" H 4707 3596 50  0000 R CNN
+F 0 "J1" H 4707 3596 50  0000 R CNN
 F 1 "Conn_ARM_JTAG_SWD_10" H 4707 3505 50  0000 R CNN
 F 2 "Connector_PinHeader_1.27mm:PinHeader_2x05_P1.27mm_Vertical_SMD" H 5150 3550 50  0001 C CNN
@@
 MCU_VDD
 $Comp
-L Connector:Conn_01x03_Female J?
+L Connector:Conn_01x03_Female J2
 U 1 1 614ABF85
 P 7550 3550
-F 0 "J?" H 7578 3576 50  0000 L CNN
+F 0 "J2" H 7578 3576 50  0000 L CNN
 F 1 "3.3V" H 7578 3485 50  0000 L CNN
 F 2 "Connector_PinHeader_2.54mm:PinHeader_1x03_P2.54mm_Vertical" H 7550 3550 50  0001 C CNN
